File: AmigaPCDriveAdapter.kicad_pcb (KiCad board)
At the start: 2 copper layers, 99.1 x 30.5 mm, 19 parts, among them P1 CONN_01X04, P2 CONN_01X04, U1 74LS38

Commit message: Correct some libraries issues. Part TWO
Parts:
- D1: footprint LEDs:LED_0603 -> LEDs:LED_1206
- R1, R2, R3, R4, R5, R6, R7, R8: footprint Resistors_SMD:R_0603_HandSoldering -> Resistors_SMD:R_1206_HandSoldering
- TO_AMIGA1: footprint Connect:IDC_Header_Straight_34pins -> RetroBitLab:IDC-Header_2x17_P2.54mm_Vertical_Lock
- turned TO_AMIGA1 to 90 degrees
Routing:
- added copper zone on F.Cu, net GND
Other:
- board text added: "designed by R.G.2018/19"
- board text removed: "designed by R.G.2018"
