File: AmigaPCDriveAdapter.sch (KiCad schematic (older format))
At the start: 18 parts, among them P1 CONN_01X04, P2 CONN_01X04, U1 74LS38

Commit message: Update libraries
Parts:
- U1: symbol 74LS38 -> 74LS38-RESCUE-AmigaPCDriveAdapter
Changed lines of the file:
@@
 EESchema Schematic File Version 2
+LIBS:AmigaPCDriveAdapter-rescue
 LIBS:power
 LIBS:device
@@
 LIBS:contrib
 LIBS:valves
+LIBS:AmigaComponents
+LIBS:4xxx
+LIBS:4xxx_IEEE
+LIBS:74xGxx
+LIBS:74xx_IEEE
+LIBS:Amplifier_Audio
+LIBS:Amplifier_Buffer
+LIBS:Amplifier_Current
+LIBS:Amplifier_Difference
+LIBS:Amplifier_Instrumentation
+LIBS:Amplifier_Operational
+LIBS:Amplifier_Video
+LIBS:Analog
+LIBS:Analog_ADC
+LIBS:Analog_DAC
+LIBS:Analog_Switch
+LIBS:Audio
+LIBS:Battery_Management
+LIBS:Comparator
+LIBS:Connector
+LIBS:Connector_Generic
+LIBS:Connector_Generic_MountingPin
+LIBS:Connector_Generic_Shielded
+LIBS:Converter_ACDC
+LIBS:Converter_DCDC
+LIBS:CPLD_Altera
+LIBS:CPLD_Xilinx
+LIBS:CPU
+LIBS:CPU_NXP_6800
+LIBS:CPU_NXP_68000
+LIBS:CPU_PowerPC
+LIBS:Device
+LIBS:Diode
+LIBS:Diode_Bridge
+LIBS:Diode_Laser
+LIBS:Display_Character
+LIBS:Display_Graphic
+LIBS:Driver_Display
+LIBS:Driver_FET
+LIBS:Driver_LED
+LIBS:Driver_Motor
+LIBS:Driver_Relay
+LIBS:DSP_AnalogDevices
+LIBS:DSP_Freescale
+LIBS:DSP_Microchip_DSPIC33
+LIBS:DSP_Motorola
+LIBS:DSP_Texas
+LIBS:Fiber_Optic
+LIBS:Filter
+LIBS:FPGA_Lattice
+LIBS:FPGA_Microsemi
+LIBS:FPGA_Xilinx
+LIBS:FPGA_Xilinx_Artix7
+LIBS:FPGA_Xilinx_Kintex7
+LIBS:FPGA_Xilinx_Spartan6
+LIBS:FPGA_Xilinx_Virtex5
+LIBS:FPGA_Xilinx_Virtex6
+LIBS:FPGA_Xilinx_Virtex7
+LIBS:ft232rl
+LIBS:GPU
+LIBS:Graphic
+LIBS:Interface
+LIBS:Interface_CAN_LIN
+LIBS:Interface_CurrentLoop
+LIBS:Interface_Ethernet
+LIBS:Interface_Expansion
+LIBS:Interface_HID
+LIBS:Interface_LineDriver
+LIBS:Interface_Optical
+LIBS:Interface_Telecom
+LIBS:Interface_UART
+LIBS:Interface_USB
+LIBS:Isolator
+LIBS:Isolator_Analog
+LIBS:Jumper
+LIBS:LED
+LIBS:Logic_LevelTranslator
+LIBS:Logic_Programmable
+LIBS:MCU_AnalogDevices
+LIBS:MCU_Cypress
+LIBS:MCU_Espressif
+LIBS:MCU_Intel
+LIBS:MCU_Microchip_8051
+LIBS:MCU_Microchip_ATmega
+LIBS:MCU_Microchip_ATtiny
+LIBS:MCU_Microchip_AVR
+LIBS:MCU_Microchip_PIC10
+LIBS:MCU_Microchip_PIC12
+LIBS:MCU_Microchip_PIC16
+LIBS:MCU_Microchip_PIC18
+LIBS:MCU_Microchip_PIC24
+LIBS:MCU_Microchip_PIC32
+LIBS:MCU_Microchip_SAMD
+LIBS:MCU_Microchip_SAME
+LIBS:MCU_Microchip_SAML
+LIBS:MCU_Module
+LIBS:MCU_Nordic
+LIBS:MCU_NXP_ColdFire
+LIBS:MCU_NXP_HC11
+LIBS:MCU_NXP_HC12
+LIBS:MCU_NXP_HCS12
+LIBS:MCU_NXP_Kinetis
+LIBS:MCU_NXP_LPC
+LIBS:MCU_NXP_MAC7100
+LIBS:MCU_NXP_MCore
+LIBS:MCU_NXP_S08
+LIBS:MCU_Parallax
+LIBS:MCU_SiFive
+LIBS:MCU_SiliconLabs
+LIBS:MCU_ST_STM8
+LIBS:MCU_ST_STM32F0
+LIBS:MCU_ST_STM32F1
+LIBS:MCU_ST_STM32F2
+LIBS:MCU_ST_STM32F3
+LIBS:MCU_ST_STM32F4
+LIBS:MCU_ST_STM32F7
+LIBS:MCU_ST_STM32H7
+LIBS:MCU_ST_STM32L0
+LIBS:MCU_ST_STM32L1
+LIBS:MCU_ST_STM32L4
+LIBS:MCU_ST_STM32L4+
+LIBS:MCU_Texas
+LIBS:MCU_Texas_MSP430
+LIBS:Mechanical
+LIBS:Memory_Controller
+LIBS:Memory_EEPROM
+LIBS:Memory_EPROM
+LIBS:Memory_Flash
+LIBS:Memory_NVRAM
+LIBS:Memory_RAM
+LIBS:Memory_ROM
+LIBS:Memory_UniqueID
+LIBS:Motor
+LIBS:Oscillator
+LIBS:Potentiometer_Digital
+LIBS:Power_Management
+LIBS:Power_Protection
+LIBS:Power_Supervisor
+LIBS:pspice
+LIBS:Reference_Current
+LIBS:Reference_Voltage
+LIBS:Regulator_Controller
+LIBS:Regulator_Current
+LIBS:Regulator_Linear
+LIBS:Regulator_SwitchedCapacitor
+LIBS:Regulator_Switching
+LIBS:Relay
+LIBS:Relay_SolidState
+LIBS:RF
+LIBS:RF_AM_FM
+LIBS:RF_Amplifier
+LIBS:RF_Bluetooth
+LIBS:RF_GPS
+LIBS:RF_GSM
+LIBS:RF_Mixer
+LIBS:RF_Module
+LIBS:RF_RFID
+LIBS:RF_Switch
+LIBS:RF_WiFi
+LIBS:RF_ZigBee
+LIBS:Security
+LIBS:Sensor
+LIBS:Sensor_Audio
+LIBS:Sensor_Current
+LIBS:Sensor_Gas
+LIBS:Sensor_Humidity
+LIBS:Sensor_Magnetic
+LIBS:Sensor_Motion
+LIBS:Sensor_Optical
+LIBS:Sensor_Pressure
+LIBS:Sensor_Proximity
+LIBS:Sensor_Temperature
+LIBS:Sensor_Touch
+LIBS:Sensor_Voltage
+LIBS:Switch
+LIBS:Timer
+LIBS:Timer_PLL
+LIBS:Timer_RTC
+LIBS:Transformer
+LIBS:Transistor_Array
+LIBS:Transistor_BJT
+LIBS:Transistor_FET
+LIBS:Transistor_IGBT
+LIBS:Triac_Thyristor
+LIBS:Valve
+LIBS:Video
 LIBS:AmigaPCDriveAdapter-cache
 EELAYER 25 0
@@
 $EndDescr
 $Comp
-L 74LS38 U1
+L 74LS38-RESCUE-AmigaPCDriveAdapter U1
 U 1 1 5BF30922
 P 4950 5900
@@
 $EndComp
 $Comp
-L 74LS38 U1
+L 74LS38-RESCUE-AmigaPCDriveAdapter U1
 U 2 1 5BF3096B
 P 5700 5800
@@
 $EndComp
 $Comp
-L 74LS38 U1
+L 74LS38-RESCUE-AmigaPCDriveAdapter U1
 U 5 1 5BF3627C
 P 3550 6300
@@
 $EndComp
 $Comp
-L 74LS38 U1
+L 74LS38-RESCUE-AmigaPCDriveAdapter U1
 U 3 1 5BF36E85
 P 4650 6650
@@
 $EndComp
 $Comp
-L 74LS38 U1
+L 74LS38-RESCUE-AmigaPCDriveAdapter U1
 U 4 1 5BF36ECC
 P 5550 6700

Commit message: Correct some libraries issues. Part TWO
Parts:
- TO_AMIGA1: footprint Connect:IDC_Header_Straight_34pins -> RetroBitLab:IDC-Header_2x17_P2.54mm_Vertical_Lock
- U1: symbol 74LS38-RESCUE-AmigaPCDriveAdapter -> AmigaPCDriveAdapter-rescue_74LS38-RESCUE-AmigaPCDriveAdapter
Changed lines of the file:
@@
 EESchema Schematic File Version 2
-LIBS:AmigaPCDriveAdapter-rescue
+LIBS:74xgxx
+LIBS:74xx
+LIBS:ac-dc
+LIBS:actel
+LIBS:adc-dac
+LIBS:Altera
+LIBS:analog_devices
+LIBS:analog_switches
+LIBS:atmel
+LIBS:audio
+LIBS:brooktre
+LIBS:cmos4000
+LIBS:cmos_ieee
+LIBS:conn
+LIBS:contrib
+LIBS:cypress
+LIBS:dc-dc
+LIBS:device
+LIBS:digital-audio
+LIBS:diode
+LIBS:display
+LIBS:dsp
+LIBS:elec-unifil
+LIBS:ESD_Protection
+LIBS:ftdi
+LIBS:gennum
+LIBS:graphic
+LIBS:hc11
+LIBS:intel
+LIBS:interface
+LIBS:ir
+LIBS:Lattice
+LIBS:linear
+LIBS:logo
+LIBS:maxim
+LIBS:memory
+LIBS:microchip
+LIBS:microchip_dspic33dsc
+LIBS:microchip_pic10mcu
+LIBS:microchip_pic12mcu
+LIBS:microchip_pic16mcu
+LIBS:microchip_pic18mcu
+LIBS:microchip_pic32mcu
+LIBS:microcontrollers
+LIBS:motor_drivers
+LIBS:motorola
+LIBS:msp430
+LIBS:nordicsemi
+LIBS:nxp_armmcu
+LIBS:onsemi
+LIBS:opto
+LIBS:Oscillators
+LIBS:philips
 LIBS:power
-LIBS:device
+LIBS:powerint
+LIBS:Power_Management
+LIBS:pspice
+LIBS:references
+LIBS:regul
+LIBS:relays
+LIBS:rfcom
+LIBS:sensors
+LIBS:silabs
+LIBS:siliconi
+LIBS:stm8
+LIBS:stm32
+LIBS:supertex
+LIBS:switches
+LIBS:texas
+LIBS:transf
 LIBS:transistors
-LIBS:conn
-LIBS:linear
-LIBS:regul
-LIBS:74xx
-LIBS:cmos4000
-LIBS:adc-dac
-LIBS:memory
+LIBS:ttl_ieee
+LIBS:valves
+LIBS:video
+LIBS:Worldsemi
+LIBS:Xicor
 LIBS:xilinx
-LIBS:microcontrollers
-LIBS:dsp
-LIBS:microchip
-LIBS:analog_switches
-LIBS:motorola
-LIBS:texas
-LIBS:intel
-LIBS:audio
-LIBS:interface
-LIBS:digital-audio
-LIBS:philips
-LIBS:display
-LIBS:cypress
-LIBS:siliconi
-LIBS:opto
-LIBS:atmel
-LIBS:contrib
-LIBS:valves
-LIBS:AmigaComponents
+LIBS:Zilog
 LIBS:4xxx
 LIBS:4xxx_IEEE
@@
 LIBS:CPU_NXP_6800
 LIBS:CPU_NXP_68000
+LIBS:CPU_NXP_IMX
 LIBS:CPU_PowerPC
 LIBS:Device
@@
 LIBS:Driver_Display
 LIBS:Driver_FET
+LIBS:Driver_Haptic
 LIBS:Driver_LED
 LIBS:Driver_Motor
@@
 LIBS:Oscillator
 LIBS:Potentiometer_Digital
-LIBS:Power_Management
 LIBS:Power_Protection
 LIBS:Power_Supervisor
-LIBS:pspice
 LIBS:Reference_Current
 LIBS:Reference_Voltage
@@
 LIBS:RF_Amplifier
 LIBS:RF_Bluetooth
+LIBS:RF_Filter
 LIBS:RF_GPS
 LIBS:RF_GSM
@@
 LIBS:Sensor_Touch
 LIBS:Sensor_Voltage
+LIBS:Simulation_SPICE
 LIBS:Switch
 LIBS:Timer
@@
 $EndDescr
 $Comp
-L 74LS38-RESCUE-AmigaPCDriveAdapter U1
+L AmigaPCDriveAdapter-rescue_74LS38-RESCUE-AmigaPCDriveAdapter U1
 U 1 1 5BF30922
 P 4950 5900
@@
 $EndComp
 $Comp
-L 74LS38-RESCUE-AmigaPCDriveAdapter U1
+L AmigaPCDriveAdapter-rescue_74LS38-RESCUE-AmigaPCDriveAdapter U1
 U 2 1 5BF3096B
 P 5700 5800
@@
 F 0 "TO_AMIGA1" V 5750 4400 50  0000 C CNN
 F 1 "CONN_02X17" V 6150 4400 50  0000 C CNN
-F 2 "Connect:IDC_Header_Straight_34pins" H 6150 3300 50  0001 C CNN
+F 2 "RetroBitLab:IDC-Header_2x17_P2.54mm_Vertical_Lock" H 6150 3300 50  0001 C CNN
 F 3 "" H 6150 3300 50  0000 C CNN
 	1    6150 4400
@@
 $EndComp
 $Comp
-L 74LS38-RESCUE-AmigaPCDriveAdapter U1
+L AmigaPCDriveAdapter-rescue_74LS38-RESCUE-AmigaPCDriveAdapter U1
 U 5 1 5BF3627C
 P 3550 6300
@@
 $EndComp
 $Comp
-L 74LS38-RESCUE-AmigaPCDriveAdapter U1
+L AmigaPCDriveAdapter-rescue_74LS38-RESCUE-AmigaPCDriveAdapter U1
 U 3 1 5BF36E85
 P 4650 6650
@@
 $EndComp
 $Comp
-L 74LS38-RESCUE-AmigaPCDriveAdapter U1
+L AmigaPCDriveAdapter-rescue_74LS38-RESCUE-AmigaPCDriveAdapter U1
 U 4 1 5BF36ECC
 P 5550 6700
@@
 Connection ~ 6600 5000
 Wire Wire Line
-	4650 1650 4650 1550
-Wire Wire Line
-	4650 1550 3850 1550
+	4650 1550 4650 1650
+Wire Wire Line
+	3850 1550 4650 1550
 Wire Wire Line
 	3850 1550 3850 1650
 Connection ~ 4100 1550
 Wire Wire Line
-	4400 1650 4400 1550
+	4400 1550 4400 1650
 Connection ~ 4400 1550
 Wire Wire Line
@@
 Connection ~ 8250 3150
 Wire Wire Line
-	8400 3150 6400 3150
+	6400 3150 8400 3150
 Connection ~ 6400 3150
 Wire Wire Line
-	5500 3150 5900 3150
+	5900 3150 5500 3150
 Connection ~ 5900 3150
 Wire Wire Line
