File: AmigaPCDriveAdapter.sch (KiCad schematic (older format))
At the start: 18 parts, among them P1 CONN_01X04, P2 CONN_01X04, U1 74LS38

Commit message: Version Kicad 5 V2.0
Parts:
- C1, C4: footprint Capacitors_SMD:C_1206_HandSoldering -> Capacitor_Tantalum_SMD:CP_EIA-3216-12_Kemet-S; symbol CP1_Small -> AmigaPCDriveAdapter-rescue:CP1_Small-AmigaPCDriveAdapter-rescue
- C2, C3: footprint Capacitors_SMD:C_1206_HandSoldering -> Capacitor_SMD:C_1206_3216Metric_Pad1.42x1.75mm_HandSolder; symbol C_Small -> AmigaPCDriveAdapter-rescue:C_Small-Device1
- D1: footprint LEDs:LED_1206 -> LED_SMD:LED_1206_3216Metric_Pad1.42x1.75mm_HandSolder; symbol Led_Small -> AmigaPCDriveAdapter-rescue:Led_Small-AmigaPCDriveAdapter-rescue
- P1: footprint Pin_Headers:Pin_Header_Straight_1x04 -> Connector_PinHeader_2.54mm:PinHeader_1x04_P2.54mm_Vertical; symbol CONN_01X04 -> AmigaPCDriveAdapter-rescue:CONN_01X04-AmigaPCDriveAdapter-rescue
- P2: footprint Pin_Headers:Pin_Header_Angled_1x04 -> Connector_PinHeader_2.54mm:PinHeader_1x04_P2.54mm_Horizontal; symbol CONN_01X04 -> AmigaPCDriveAdapter-rescue:CONN_01X04-AmigaPCDriveAdapter-rescue
- R1, R2, R3, R4, R5, R6, R7, R8: footprint Resistors_SMD:R_1206_HandSoldering -> Resistor_SMD:R_1206_3216Metric_Pad1.42x1.75mm_HandSolder; symbol R -> AmigaPCDriveAdapter-rescue:R-AmigaPCDriveAdapter-rescue
- TO_AMIGA1: symbol CONN_02X17 -> AmigaPCDriveAdapter-rescue:CONN_02X17-AmigaPCDriveAdapter-rescue
- TO_FLOPPY1: footprint Socket_Strips:Socket_Strip_Straight_2x17 -> Connector_PinSocket_2.54mm:PinSocket_2x17_P2.54mm_Vertical; symbol CONN_02X17 -> AmigaPCDriveAdapter-rescue:CONN_02X17-AmigaPCDriveAdapter-rescue
- U1: footprint Housings_DIP:DIP-14_W7.62mm -> Package_DIP:DIP-14_W7.62mm; symbol AmigaPCDriveAdapter-rescue_74LS38-RESCUE-AmigaPCDriveAdapter -> AmigaPCDriveAdapter-rescue:AmigaPCDriveAdapter-rescue_74LS38-RESCUE-AmigaPCDriveAdapter-AmigaPCDriveAdapter-rescue
Connections:
- wire segments 78 -> 127

Commit message: Updated to drop the rescue file
Parts:
- C1, C4: symbol AmigaPCDriveAdapter-rescue:CP1_Small-AmigaPCDriveAdapter-rescue -> Device:CP1_Small
- C2, C3: symbol AmigaPCDriveAdapter-rescue:C_Small-Device1 -> Device:C_Small
- D1: symbol AmigaPCDriveAdapter-rescue:Led_Small-AmigaPCDriveAdapter-rescue -> Device:LED_Small
- P1, P2: symbol AmigaPCDriveAdapter-rescue:CONN_01X04-AmigaPCDriveAdapter-rescue -> Connector_Generic:Conn_01x04
- R1, R2, R3, R4, R5, R6, R7, R8: symbol AmigaPCDriveAdapter-rescue:R-AmigaPCDriveAdapter-rescue -> Device:R
- TO_AMIGA1, TO_FLOPPY1: symbol AmigaPCDriveAdapter-rescue:CONN_02X17-AmigaPCDriveAdapter-rescue -> Connector_Generic:Conn_02x17_Odd_Even
- U1: symbol AmigaPCDriveAdapter-rescue:AmigaPCDriveAdapter-rescue_74LS38-RESCUE-AmigaPCDriveAdapter-AmigaPCDriveAdapter-rescue -> 74xx:74LS38
Changed lines of the file:
@@
 $EndDescr
 $Comp
-L AmigaPCDriveAdapter-rescue:AmigaPCDriveAdapter-rescue_74LS38-RESCUE-AmigaPCDriveAdapter-AmigaPCDriveAdapter-rescue U1
+L 74xx:74LS38 U1
 U 1 1 5BF30922
 P 4950 5900
@@
 $EndComp
 $Comp
-L AmigaPCDriveAdapter-rescue:AmigaPCDriveAdapter-rescue_74LS38-RESCUE-AmigaPCDriveAdapter-AmigaPCDriveAdapter-rescue U1
+L 74xx:74LS38 U1
 U 2 1 5BF3096B
 P 5700 5800
@@
 $EndComp
 $Comp
-L AmigaPCDriveAdapter-rescue:CONN_02X17-AmigaPCDriveAdapter-rescue TO_FLOPPY1
+L Connector_Generic:Conn_02x17_Odd_Even TO_FLOPPY1
 U 1 1 5BF325B4
-P 6150 1950
-F 0 "TO_FLOPPY1" V 5750 1900 50  0000 C CNN
-F 1 "CONN_02X17" V 6150 1950 50  0000 C CNN
-F 2 "Connector_PinSocket_2.54mm:PinSocket_2x17_P2.54mm_Vertical" H 6150 850 50  0001 C CNN
-F 3 "" H 6150 850 50  0000 C CNN
-	1    6150 1950
-	1    0    0    -1
-$EndComp
-$Comp
-L AmigaPCDriveAdapter-rescue:CONN_02X17-AmigaPCDriveAdapter-rescue TO_AMIGA1
+P 6100 1950
+F 0 "TO_FLOPPY1" V 5700 1900 50  0000 C CNN
+F 1 "CONN_02X17" V 6100 1950 50  0000 C CNN
+F 2 "Connector_PinSocket_2.54mm:PinSocket_2x17_P2.54mm_Vertical" H 6100 850 50  0001 C CNN
+F 3 "" H 6100 850 50  0000 C CNN
+	1    6100 1950
+	1    0    0    -1
+$EndComp
+$Comp
+L Connector_Generic:Conn_02x17_Odd_Even TO_AMIGA1
 U 1 1 5BF32608
-P 6150 4400
-F 0 "TO_AMIGA1" V 5750 4400 50  0000 C CNN
-F 1 "CONN_02X17" V 6150 4400 50  0000 C CNN
-F 2 "RetroBitLab:IDC-Header_2x17_P2.54mm_Vertical_Lock" H 6150 3300 50  0001 C CNN
-F 3 "" H 6150 3300 50  0000 C CNN
-	1    6150 4400
+P 6100 4400
+F 0 "TO_AMIGA1" V 5700 4400 50  0000 C CNN
+F 1 "CONN_02X17" V 6100 4400 50  0000 C CNN
+F 2 "RetroBitLab:IDC-Header_2x17_P2.54mm_Vertical_Lock" H 6100 3300 50  0001 C CNN
+F 3 "" H 6100 3300 50  0000 C CNN
+	1    6100 4400
 	1    0    0    -1
 $EndComp
 NoConn ~ 6400 1150
 $Comp
-L AmigaPCDriveAdapter-rescue:GND-power1 #PWR01
+L power:GND #PWR01
 U 1 1 5BF336B1
 P 5500 3300
@@
 $EndComp
 $Comp
-L AmigaPCDriveAdapter-rescue:PWR_FLAG-power1 #FLG02
+L power:PWR_FLAG #FLG02
 U 1 1 5BF336CD
 P 5500 3150
@@
 $EndComp
 $Comp
-L AmigaPCDriveAdapter-rescue:R-AmigaPCDriveAdapter-rescue R7
+L Device:R R7
 U 1 1 5BF33A10
 P 6600 5650
@@
 $EndComp
 $Comp
-L AmigaPCDriveAdapter-rescue:+5V-power1 #PWR03
+L power:+5V #PWR03
 U 1 1 5BF33AD3
 P 6600 5500
@@
 $EndComp
 $Comp
-L AmigaPCDriveAdapter-rescue:PWR_FLAG-power1 #FLG04
+L power:PWR_FLAG #FLG04
 U 1 1 5BF33C2A
 P 6600 5500
@@
 ~REDWC
 $Comp
-L AmigaPCDriveAdapter-rescue:R-AmigaPCDriveAdapter-rescue R6
+L Device:R R6
 U 1 1 5BF33E24
 P 8250 2950
@@
 $EndComp
 $Comp
-L AmigaPCDriveAdapter-rescue:+5V-power1 #PWR05
+L power:+5V #PWR05
 U 1 1 5BF33E57
 P 8250 2800
@@
 $EndComp
 $Comp
-L AmigaPCDriveAdapter-rescue:R-AmigaPCDriveAdapter-rescue R5
+L Device:R R5
 U 1 1 5BF33E87
 P 5250 6050
@@
 $EndComp
 $Comp
-L AmigaPCDriveAdapter-rescue:+5V-power1 #PWR06
+L power:+5V #PWR06
 U 1 1 5BF33F39
 P 5250 6200
@@
 ~INDEX
 $Comp
-L AmigaPCDriveAdapter-rescue:+5V-power1 #PWR07
+L power:+5V #PWR07
 U 1 1 5BF34B97
 P 4250 1300
@@
 $EndComp
 $Comp
-L AmigaPCDriveAdapter-rescue:R-AmigaPCDriveAdapter-rescue R4
+L Device:R R4
 U 1 1 5BF351BE
 P 4650 1800
@@
 $EndComp
 $Comp
-L AmigaPCDriveAdapter-rescue:R-AmigaPCDriveAdapter-rescue R3
+L Device:R R3
 U 1 1 5BF35267
 P 4400 1800
@@
 $EndComp
 $Comp
-L AmigaPCDriveAdapter-rescue:R-AmigaPCDriveAdapter-rescue R2
+L Device:R R2
 U 1 1 5BF35298
 P 4100 1800
@@
 $EndComp
 $Comp
-L AmigaPCDriveAdapter-rescue:R-AmigaPCDriveAdapter-rescue R1
+L Device:R R1
 U 1 1 5BF352CE
 P 3850 1800
@@
 $EndComp
 $Comp
-L AmigaPCDriveAdapter-rescue:CONN_01X04-AmigaPCDriveAdapter-rescue P1
+L Connector_Generic:Conn_01x04 P1
 U 1 1 5BF353AC
-P 2750 3350
-F 0 "P1" H 2750 3600 50  0000 C CNN
-F 1 "CONN_01X04" V 2850 3350 50  0000 C CNN
-F 2 "Connector_PinHeader_2.54mm:PinHeader_1x04_P2.54mm_Vertical" H 2750 3350 50  0001 C CNN
-F 3 "" H 2750 3350 50  0000 C CNN
-	1    2750 3350
+P 2800 3350
+F 0 "P1" H 2800 3600 50  0000 C CNN
+F 1 "CONN_01X04" V 2900 3350 50  0000 C CNN
+F 2 "Connector_PinHeader_2.54mm:PinHeader_1x04_P2.54mm_Vertical" H 2800 3350 50  0001 C CNN
+F 3 "" H 2800 3350 50  0000 C CNN
+	1    2800 3350
 	0    1    1    0
 $EndComp
 $Comp
-L AmigaPCDriveAdapter-rescue:+5V-power1 #PWR08
+L power:+5V #PWR08
 U 1 1 5BF355B6
 P 2900 2950
@@
 $EndComp
 $Comp
-L AmigaPCDriveAdapter-rescue:+12V-power1 #PWR09
+L power:+12V #PWR09
 U 1 1 5BF355E2
 P 2600 2950
@@
 $EndComp
 $Comp
-L AmigaPCDriveAdapter-rescue:GND-power1 #PWR010
+L power:GND #PWR010
 U 1 1 5BF3560E
 P 2700 3150
@@
 $EndComp
 $Comp
-L AmigaPCDriveAdapter-rescue:GND-power1 #PWR011
+L power:GND #PWR011
 U 1 1 5BF35644
 P 2800 3150
@@
 $EndComp
 $Comp
-L AmigaPCDriveAdapter-rescue:PWR_FLAG-power1 #FLG012
+L power:PWR_FLAG #FLG012
 U 1 1 5BF35673
 P 2600 2950
@@
 $EndComp
 $Comp
-L AmigaPCDriveAdapter-rescue:CONN_01X04-AmigaPCDriveAdapter-rescue P2
+L Connector_Generic:Conn_01x04 P2
 U 1 1 5BF35EC9
-P 1400 3350
-F 0 "P2" H 1400 3600 50  0000 C CNN
-F 1 "CONN_01X04" V 1500 3350 50  0000 C CNN
-F 2 "Connector_PinHeader_2.54mm:PinHeader_1x04_P2.54mm_Horizontal" H 1400 3350 50  0001 C CNN
-F 3 "" H 1400 3350 50  0000 C CNN
-	1    1400 3350
+P 1450 3350
+F 0 "P2" H 1450 3600 50  0000 C CNN
+F 1 "CONN_01X04" V 1550 3350 50  0000 C CNN
+F 2 "Connector_PinHeader_2.54mm:PinHeader_1x04_P2.54mm_Horizontal" H 1450 3350 50  0001 C CNN
+F 3 "" H 1450 3350 50  0000 C CNN
+	1    1450 3350
 	0    1    1    0
 $EndComp
 $Comp
-L AmigaPCDriveAdapter-rescue:+5V-power1 #PWR013
+L power:+5V #PWR013
 U 1 1 5BF35ED1
 P 1550 2950
@@
 $EndComp
 $Comp
-L AmigaPCDriveAdapter-rescue:+12V-power1 #PWR014
+L power:+12V #PWR014
 U 1 1 5BF35ED7
 P 1250 2950
@@
 $EndComp
 $Comp
-L AmigaPCDriveAdapter-rescue:GND-power1 #PWR015
+L power:GND #PWR015
 U 1 1 5BF35EDD
 P 1350 3150
@@
 $EndComp
 $Comp
-L AmigaPCDriveAdapter-rescue:GND-power1 #PWR016
+L power:GND #PWR016
 U 1 1 5BF35EE3
 P 1450 3150
@@
 $EndComp
 $Comp
-L AmigaPCDriveAdapter-rescue:AmigaPCDriveAdapter-rescue_74LS38-RESCUE-AmigaPCDriveAdapter-AmigaPCDriveAdapter-rescue U1
+L 74xx:74LS38 U1
 U 5 1 5BF3627C
 P 3550 6300
@@
 $EndComp
 $Comp
-L AmigaPCDriveAdapter-rescue:+5V-power1 #PWR017
+L power:+5V #PWR017
 U 1 1 5BF36319
 P 3550 5800
@@
 $EndComp
 $Comp
-L AmigaPCDriveAdapter-rescue:GND-power1 #PWR018
+L power:GND #PWR018
 U 1 1 5BF3636C
 P 3550 6800
@@
 $EndComp
 $Comp
-L AmigaPCDriveAdapter-rescue:AmigaPCDriveAdapter-rescue_74LS38-RESCUE-AmigaPCDriveAdapter-AmigaPCDriveAdapter-rescue U1
+L 74xx:74LS38 U1
 U 3 1 5BF36E85
 P 4650 6650
@@
 $EndComp
 $Comp
-L AmigaPCDriveAdapter-rescue:AmigaPCDriveAdapter-rescue_74LS38-RESCUE-AmigaPCDriveAdapter-AmigaPCDriveAdapter-rescue U1
+L 74xx:74LS38 U1
 U 4 1 5BF36ECC
 P 5550 6700
@@
 NoConn ~ 4350 6550
 $Comp
-L AmigaPCDriveAdapter-rescue:GND-power1 #PWR019
+L power:GND #PWR019
 U 1 1 5BF37D1F
 P 2900 1900
@@
 $EndComp
 $Comp
-L AmigaPCDriveAdapter-rescue:+5V-power1 #PWR020
+L power:+5V #PWR020
 U 1 1 5BF37D71
 P 2900 1400
@@
 $EndComp
 $Comp
-L AmigaPCDriveAdapter-rescue:R-AmigaPCDriveAdapter-rescue R8
+L Device:R R8
 U 1 1 5BF37D9E
 P 2900 1550
@@
 $EndComp
 $Comp
-L AmigaPCDriveAdapter-rescue:Led_Small-AmigaPCDriveAdapter-rescue D1
+L Device:LED_Small D1
 U 1 1 5BF37DE7
 P 2900 1800
@@
 $EndComp
 $Comp
-L AmigaPCDriveAdapter-rescue:+12V-power1 #PWR021
+L power:+12V #PWR021
 U 1 1 5C1F99AB
 P 1400 1350
@@
 $EndComp
 $Comp
-L AmigaPCDriveAdapter-rescue:GND-power1 #PWR022
+L power:GND #PWR022
 U 1 1 5C1F99EC
 P 1400 1900
@@
 $EndComp
 $Comp
-L AmigaPCDriveAdapter-rescue:C_Small-Device1 C2
+L Device:C_Small C2
 U 1 1 5C1F9A1D
 P 1400 1600
@@
 $EndComp
 $Comp
-L AmigaPCDriveAdapter-rescue:C_Small-Device1 C3
+L Device:C_Small C3
 U 1 1 5C1F9A72
 P 1950 1600
@@
 $EndComp
 $Comp
-L AmigaPCDriveAdapter-rescue:+5V-power1 #PWR023
+L power:+5V #PWR023
 U 1 1 5C1F9B0B
 P 1950 1350
@@
 $EndComp
 $Comp
-L AmigaPCDriveAdapter-rescue:GND-power1 #PWR024
+L power:GND #PWR024
 U 1 1 5C1F9B52
 P 1950 1900
@@
 $EndComp
 $Comp
-L AmigaPCDriveAdapter-rescue:CP1_Small-AmigaPCDriveAdapter-rescue C4
+L Device:CP1_Small C4
 U 1 1 5C1F9BAF
 P 2350 1600
@@
 $EndComp
 $Comp
-L AmigaPCDriveAdapter-rescue:CP1_Small-AmigaPCDriveAdapter-rescue C1
+L Device:CP1_Small C1
 U 1 1 5C1F9BF4
 P 950 1600

Commit message: Generated with latest version of KiCAD 5.1.9
Parts:
- C2, C3: footprint Capacitor_SMD:C_1206_3216Metric_Pad1.42x1.75mm_HandSolder -> Capacitor_SMD:C_1206_3216Metric_Pad1.33x1.80mm_HandSolder
- R1, R2, R3, R4, R5, R6, R7, R8: footprint Resistor_SMD:R_1206_3216Metric_Pad1.42x1.75mm_HandSolder -> Resistor_SMD:R_1206_3216Metric_Pad1.30x1.75mm_HandSolder
Changed lines of the file:
@@
 EESchema Schematic File Version 4
-LIBS:AmigaPCDriveAdapter-cache
-EELAYER 26 0
+EELAYER 30 0
 EELAYER END
 $Descr A4 11693 8268
@@
 Sheet 1 1
 Title "AMIGA PC FLOPPY ADAPTER"
-Date "2021-01-23"
-Rev "2.0"
+Date "2022-04-01"
+Rev "2.1"
 Comp "RETROBIT LAB"
 Comment1 "Gianluca Renzi <icjtqr@gmail.com>"
@@
 F 0 "R7" V 6680 5650 50  0000 C CNN
 F 1 "2.2K" V 6600 5650 50  0000 C CNN
-F 2 "Resistor_SMD:R_1206_3216Metric_Pad1.42x1.75mm_HandSolder" V 6530 5650 50  0001 C CNN
+F 2 "Resistor_SMD:R_1206_3216Metric_Pad1.30x1.75mm_HandSolder" V 6530 5650 50  0001 C CNN
 F 3 "" H 6600 5650 50  0000 C CNN
 	1    6600 5650
@@
 F 0 "R6" V 8330 2950 50  0000 C CNN
 F 1 "2,2K" V 8250 2950 50  0000 C CNN
-F 2 "Resistor_SMD:R_1206_3216Metric_Pad1.42x1.75mm_HandSolder" V 8180 2950 50  0001 C CNN
+F 2 "Resistor_SMD:R_1206_3216Metric_Pad1.30x1.75mm_HandSolder" V 8180 2950 50  0001 C CNN
 F 3 "" H 8250 2950 50  0000 C CNN
 	1    8250 2950
@@
 F 0 "R5" V 5330 6050 50  0000 C CNN
 F 1 "2.2K" V 5250 6050 50  0000 C CNN
-F 2 "Resistor_SMD:R_1206_3216Metric_Pad1.42x1.75mm_HandSolder" V 5180 6050 50  0001 C CNN
+F 2 "Resistor_SMD:R_1206_3216Metric_Pad1.30x1.75mm_HandSolder" V 5180 6050 50  0001 C CNN
 F 3 "" H 5250 6050 50  0000 C CNN
 	1    5250 6050
@@
 F 0 "R4" V 4730 1800 50  0000 C CNN
 F 1 "2.2K" V 4650 1800 50  0000 C CNN
-F 2 "Resistor_SMD:R_1206_3216Metric_Pad1.42x1.75mm_HandSolder" V 4580 1800 50  0001 C CNN
+F 2 "Resistor_SMD:R_1206_3216Metric_Pad1.30x1.75mm_HandSolder" V 4580 1800 50  0001 C CNN
 F 3 "" H 4650 1800 50  0000 C CNN
 	1    4650 1800
@@
 F 0 "R3" V 4480 1800 50  0000 C CNN
 F 1 "2.2K" V 4400 1800 50  0000 C CNN
-F 2 "Resistor_SMD:R_1206_3216Metric_Pad1.42x1.75mm_HandSolder" V 4330 1800 50  0001 C CNN
+F 2 "Resistor_SMD:R_1206_3216Metric_Pad1.30x1.75mm_HandSolder" V 4330 1800 50  0001 C CNN
 F 3 "" H 4400 1800 50  0000 C CNN
 	1    4400 1800
@@
 F 0 "R2" V 4180 1800 50  0000 C CNN
 F 1 "2.2K" V 4100 1800 50  0000 C CNN
-F 2 "Resistor_SMD:R_1206_3216Metric_Pad1.42x1.75mm_HandSolder" V 4030 1800 50  0001 C CNN
+F 2 "Resistor_SMD:R_1206_3216Metric_Pad1.30x1.75mm_HandSolder" V 4030 1800 50  0001 C CNN
 F 3 "" H 4100 1800 50  0000 C CNN
 	1    4100 1800
@@
 F 0 "R1" V 3930 1800 50  0000 C CNN
 F 1 "2.2K" V 3850 1800 50  0000 C CNN
-F 2 "Resistor_SMD:R_1206_3216Metric_Pad1.42x1.75mm_HandSolder" V 3780 1800 50  0001 C CNN
+F 2 "Resistor_SMD:R_1206_3216Metric_Pad1.30x1.75mm_HandSolder" V 3780 1800 50  0001 C CNN
 F 3 "" H 3850 1800 50  0000 C CNN
 	1    3850 1800
@@
 F 0 "R8" V 2980 1550 50  0000 C CNN
 F 1 "330" V 2900 1550 50  0000 C CNN
-F 2 "Resistor_SMD:R_1206_3216Metric_Pad1.42x1.75mm_HandSolder" V 2830 1550 50  0001 C CNN
+F 2 "Resistor_SMD:R_1206_3216Metric_Pad1.30x1.75mm_HandSolder" V 2830 1550 50  0001 C CNN
 F 3 "" H 2900 1550 50  0000 C CNN
 	1    2900 1550
@@
 F 0 "C2" H 1410 1670 50  0000 L CNN
 F 1 "100nF" H 1410 1520 50  0000 L CNN
-F 2 "Capacitor_SMD:C_1206_3216Metric_Pad1.42x1.75mm_HandSolder" H 1400 1600 50  0001 C CNN
+F 2 "Capacitor_SMD:C_1206_3216Metric_Pad1.33x1.80mm_HandSolder" H 1400 1600 50  0001 C CNN
 F 3 "" H 1400 1600 50  0000 C CNN
 	1    1400 1600
@@
 F 0 "C3" H 1960 1670 50  0000 L CNN
 F 1 "100nF" H 1960 1520 50  0000 L CNN
-F 2 "Capacitor_SMD:C_1206_3216Metric_Pad1.42x1.75mm_HandSolder" H 1950 1600 50  0001 C CNN
+F 2 "Capacitor_SMD:C_1206_3216Metric_Pad1.33x1.80mm_HandSolder" H 1950 1600 50  0001 C CNN
 F 3 "" H 1950 1600 50  0000 C CNN
 	1    1950 1600
